File: Hardware/PCB/V2/FilamentBox.sch (EAGLE design)
At the start: 25 parts, among them IC1 7805TV, Q1 BC817, Q2 NX2301P, Q3 BC817, U3 PHOTON

Commit message: Update (to 2.04)- Added reverse mount LEDs (Red, Yellow and Green for Humidity warning, fan status and OK (with OSH Logo)). Added poly fuse and diode for input protection. Swapped orientation of VIn connector and voltage regulator for better layout. Added PCB images generated by DirtyPCBs (note text is wrong way around).
Sent to DirtyPCBs (3-Jan-2017)
Parts:
- removed C3: 10uF, SparkFun-Capacitors:CAP_POLPTH2
- removed JP4: (no value), SparkFun-Connectors:M04PTH
- added C5: 0.1uF 25V, SparkFun-Capacitors:1UF-25V-10%(0805)"
- added D3: Green, SparkFun-LED:LED1206-BOTTOM
- added D4: MBRA140, SparkFun-DiscreteSemi:DIODE-SCHOTTKY-MBRA140
- added D7: Red, SparkFun-LED:LED1206-BOTTOM
- added D8: Yellow, SparkFun-LED:LED1206-BOTTOM
- added F1: SMD100F/33, switch-raychem:SMD100F/33
- added FRAME1: FRAME-LETTER, SparkFun-Aesthetics:FRAME-LETTER
- added R5, R6, R7: 1k5, SparkFun-Resistors:RESISTOR0805-RES
- C4: value 1uF -> 0.1uF 10V
- LOGO1: value OSHW-LOGOS -> OSHW-LOGOL; device Spark:OSHW-LOGOS -> Spark:OSHW-LOGOL
- SG1: FARNELL (none) -> 2098836
Connections:
- removed net N$7: JP5.4, U3.A3
- removed net N$8: JP5.5, U3.A4
- removed net N$9: JP5.6, U3.A5
- new net FAN_LED: JP5.5, R7.2, U3.A4
- new net HIGH_HUMIDITY_LED: JP5.4, R6.2, U3.A3
- new net N$18: D3.A, R5.1
- new net N$19: F1.1, JP1.2
- new net N$20: D4.A, F1.2
- new net N$25: D7.A, R6.1
- new net N$26: D8.A, R7.1
- new net OSH_LED: JP5.6, R5.2, U3.A5
- net 3.3V: no longer JP4.1
- net BUZZER: now also JP5.7, U3.DAC; no longer JP9.8, U3.D2
- net GND: now also C5.2, D3.C, D7.C, D8.C; no longer C3.-, JP4.2
- net N$10: now also JP9.8, U3.D2; no longer JP5.7, U3.DAC
- net SCL: no longer JP4.4
- net SDA: no longer JP4.3
- net VIN: now also C5.1, D4.C; no longer C3.+, JP1.2
Other:
- note added: "2.04"
- note added: "Fan Control"
- note added: "Humidity Sensor"
- note added: "Photon Controller"
- note added: "Power In."
- note added: "S.Harrison"
- note added: "Use buck switching module rather than 7805"
- note added: "Warning Buzzer"
- note removed: "For better thermal efficiency use switching module rather than 7805"
- note removed: "SparkFun HTU21D Breakout (12064)"
- moved on the sheet: C2, C4, D1, D2, IC1, JP1, JP11, JP2, JP3, JP5, JP8, JP9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

Commit message: Added part values
Parts:
- F1: FARNELL (none) -> 1822224; MFG (none) -> LITTLEFUSE; MFGPART (none) -> 2920L075DR
Changed lines of the file:
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@@
 <part name="R7" library="SparkFun-Resistors" deviceset="RESISTOR" device="0805-RES" value="1k5"/>
 <part name="GND5" library="SparkFun-Aesthetics" deviceset="GND" device=""/>
-<part name="F1" library="switch-raychem" deviceset="SMD*F" device="/33" technology="100"/>
+<part name="F1" library="switch-raychem" deviceset="SMD*F" device="/33" technology="100">
+<attribute name="FARNELL" value="1822224"/>
+<attribute name="MFG" value="LITTLEFUSE"/>
+<attribute name="MFGPART" value="2920L075DR"/>
+</part>
 <part name="D7" library="SparkFun-LED" deviceset="LED" device="1206-BOTTOM" value="Red"/>
 <part name="D8" library="SparkFun-LED" deviceset="LED" device="1206-BOTTOM" value="Yellow"/>
@@
 <text x="190.5" y="114.3" size="1.778" layer="97">Humidity Sensor</text>
 <text x="236.22" y="17.78" size="1.778" layer="97">2.04</text>
-<text x="165.1" y="20.32" size="1.778" layer="97">S.Harrison</text>
+<text x="168.402" y="21.844" size="1.778" layer="97">S.Harrison</text>
 <wire x1="0" y1="152.4" x2="66.04" y2="152.4" width="0.1524" layer="97"/>
 <wire x1="66.04" y1="152.4" x2="66.04" y2="119.38" width="0.1524" layer="97"/>
@@
 <instance part="R7" gate="G$1" x="40.64" y="129.54" rot="R180"/>
 <instance part="GND5" gate="1" x="58.42" y="124.46"/>
-<instance part="F1" gate="G$1" x="33.02" y="180.34"/>
+<instance part="F1" gate="G$1" x="33.02" y="180.34">
+<attribute name="FARNELL" x="33.02" y="180.34" size="1.27" layer="96" display="off"/>
+<attribute name="MFG" x="33.02" y="180.34" size="1.778" layer="96" display="off"/>
+<attribute name="MFGPART" x="33.02" y="180.34" size="1.778" layer="96" display="off"/>
+</instance>
 <instance part="D7" gate="G$1" x="50.8" y="142.24" rot="R90"/>
 <instance part="D8" gate="G$1" x="50.8" y="129.54" rot="R90"/>
-<instance part="LOGO1" gate="G$1" x="231.14" y="68.58"/>
+<instance part="LOGO1" gate="G$1" x="228.6" y="71.12"/>
 </instances>
 <busses>
